File: pathfinder.kicad_pcb (KiCad board)
At the start: 2 copper layers, 57.2 x 44 mm, 15 parts, among them SW1 SW_Push, SW2 SW_Push, SW3 SW_Push, SW4 SW_SPST, U1 XIAO-RP2040-SMD

Commit message: Finished arduino code
Parts:
- added D4: L08R5000Q1, e390cee6c564169ed6d49fe7a268946ec8897500_l08r5000q1:LEDRD254W57D500H1070, F.Cu at (151.7, 154.5)
- added J1: Conn_01x02_Socket, Connector_PinSocket_2.54mm:PinSocket_1x02_P2.54mm_Vertical, F.Cu at (126.2, 153.1)
- added R5: 5k, Resistor_THT:R_Axial_DIN0204_L3.6mm_D1.6mm_P5.08mm_Horizontal, F.Cu at (167.0, 143.1)
- moved D3 7.24 mm to (158.0, 154.5)
- moved D2 3.48 mm to (164.2, 154.5)
- moved R4 1.95 mm to (169.1, 143.0)
- moved R3 0.93 mm to (171.3, 143.0)
- moved D1 0.25 mm to (170.5, 154.5)
- moved R2 0.12 mm to (173.4, 143.0)
Connections:
- U1 pad 3: unconnected-(U1-GPIO28_A2_D2-Pad3) -> MOTOR
- U1 pad 8: unconnected-(U1-GPIO1_D7_CSn_RX-Pad8) -> LED4
Routing:
- net LED4: track 0.00 -> 23.2 mm, vias 0 -> 1
- net Net-(D4-PadA): track 0.00 -> 16.7 mm
- net Net-(D3-PadA): track 17.9 -> 12.5 mm
- net GND: track 4.59 -> 0.00 mm, vias 2 -> 6
- net Net-(D2-PadA): track 11.0 -> 8.83 mm
- net LED3: track 23.0 -> 25.0 mm
- net LED2: track 26.0 -> 26.9 mm
Other:
- board text added: "+ -"
