File: pathfinder.kicad_sch (KiCad schematic)
At the start: 14 parts, among them SW1 SW_Push, SW2 SW_Push, SW3 SW_Push, SW4 SW_SPST, U1 XIAO-RP2040-SMD

Commit message: Finished arduino code
Parts:
- added D4: L08R5000Q1, e390cee6c564169ed6d49fe7a268946ec8897500_l08r5000q1:LEDRD254W57D500H1070, symbol L08R5000Q1:L08R5000Q1
- added J1: Conn_01x02_Socket, Connector_PinSocket_2.54mm:PinSocket_1x02_P2.54mm_Vertical, symbol Connector:Conn_01x02_Socket
- added R5: 5k, Resistor_THT:R_Axial_DIN0204_L3.6mm_D1.6mm_P5.08mm_Horizontal, symbol Device:R
Connections:
- net GND: now also D4.C, J1.2 (Pin_2)
- net MOTOR: now reaches U1.3 (GPIO28_A2_D2)
- net MOTOR: now also J1.1 (Pin_1)
- net LED4: now reaches U1.8 (GPIO1_D7_CSn_RX)
- net LED4: now also R5.1
- new net: D4.A, R5.2
Other:
- moved on the sheet: R1
